File: elec_board/VisionIndustrielle_TP.kicad_pcb (KiCad board)
At the start: 2 copper layers, 148 x 111.1 mm, 48 parts, among them J1 Capt1, J10 Morpho_Gauche, J11 RN42X-DROITE, J12 BAT_IN, J13 Motor1_Out_JST, J14 Morpho_Droite, J15 Poussoir1, J16 Poussoir2, J17 Motor1_Out_Pin, J18 GND_reg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

Commit message: Update Schematic
Connections:
- J14 pad 36: Net-(J14-Pad36) -> STEP_NUC
Routing:
- net STEP_NUC: track 51.1 -> 53.6 mm
