File: elec_board/VisionIndustrielle_TP.sch (KiCad schematic (older format))
At the start: 44 parts, among them J1 Capt1, J10 Morpho_Gauche, J11 RN42X-DROITE, J12 BAT_IN, J13 Motor1_Out_JST, J14 Morpho_Droite, J15 Poussoir1, J16 Poussoir2, J17 Motor1_Out_Pin, J18 GND_reg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

Commit message: Update Schematic
Connections:
- net STEP_NUC: now also J14.36 (Pin_36)
Changed lines of the file:
@@
 Wire Wire Line
 	6150 3300 6250 3300
+Text GLabel 6250 3800 2    50   Input ~ 0
+STEP_NUC
+Wire Wire Line
+	6150 3800 6250 3800
 $EndSCHEMATC
